File: PCB_design/Circuit_Design_DO/Circuit_Design_DO.kicad_sch (KiCad schematic)
At the start: 0 parts

Commit message: Added new folder for components and initial commit of schematic work
Parts:
- added C1: 10n, symbol Device:C
- added C10, C11: 0.1u, symbol Device:C_Polarized
- added C12: 3.3n, symbol Device:C
- added C2, C9: 1u, symbol Device:C
- added C3, C6, C8: 1n, symbol Device:C
- added C4, C5, C7: 100n, symbol Device:C
- added D1: SMF5V0A, Diode_SMD:D_SMF, symbol Diode:SMF5V0A
- added J1: Conn_Coaxial, symbol Connector:Conn_Coaxial
- added J2: USB_C_Receptacle_PowerOnly_6P, symbol Connector:USB_C_Receptacle_PowerOnly_6P
- added J3: USB_C_Receptacle_USB2.0_14P, symbol Connector:USB_C_Receptacle_USB2.0_14P
- added R1, R3: 1.62M, symbol Device:R
- added R2: 47k, symbol Device:R
- added R4: 1780, symbol Device:R
- added R5, Rsns: 10k, symbol Device:R
- added R6: 332k, symbol Device:R
- added R7: 118k, symbol Device:R
- added R8, R9: 5.1k, symbol Device:R
- added U1: AMC3330, Package_SO:SOIC-16W_7.5x10.3mm_P1.27mm, symbol Isolator_Analog:AMC3330
- added U2: ADS8681RUM, Package_DFN_QFN:QFN-16-1EP_4x4mm_P0.65mm_EP2.7x2.7mm, symbol Analog_ADC:ADS8681RUM
- added U3: TPS259571DSGR, DSG0008A, symbol 2025-10-29_16-24-21:TPS259571DSGR
- added U4: ADUM3160, Package_SO:SOIC-16W_7.5x10.3mm_P1.27mm, symbol Interface_USB:ADUM3160
Connections:
- new net: C10.1, D1.1 (A1), J2.A9 (VBUS), J2.B9 (VBUS), R5.1, R6.1, U3.3 (IN), U3.4 (IN)
- new net: R6.2, R7.1, U3.2 (EN_UVLO)
- new net: C12.1, U3.1 (DV_DT)
- new net: J3.A4 (VBUS), J3.A9 (VBUS), J3.B4 (VBUS), J3.B9 (VBUS)
- new net: C1.1, R1.2, Rsns.1, U1.6 (INP)
- new net: C1.2, C2.2, C3.2, C4.2, C5.1, C6.2, R3.1, Rsns.2, U1.2 (DCDC_HGND), U1.7 (INN), U1.8 (HGND)
- new net: J2.A5 (CC1), R8.1
- new net: J2.B5 (CC2), R9.1
- new net: R4.1, U3.7 (ILM)
- new net: C7.1, U1.13 (LDO_OUT), U1.16 (DCDC_IN)
- new net: C3.1, C4.1, U1.5 (HLDO_OUT)
- new net: C2.1, C5.2, C6.1, U1.1 (DCDC_OUT), U1.3 (HLDO_IN)
- new net: J1.1 (In), R1.1
- new net: J1.2 (Ext), R3.2
- new net +5V: C11.1, C8.1, C9.1, R2.1, U1.12 (VDD), U3.5 (OUT)
- new net ADC+: U1.11 (OUTP)
- new net ADC-: U1.10 (OUTN)
- new net DIAG: R2.2, U1.14 (DIAG)
- new net FLT_eFuse: R5.2, U3.6 (FLT_N)
- new net GND: C10.2, C11.2, C12.2, C7.2, C8.2, C9.2, D1.2 (A2), J2.A12 (GND), J2.B12 (GND), J2.S1 (SHIELD), J3.A1 (GND), J3.A12 (GND), J3.B1 (GND), J3.B12 (GND), J3.S1 (SHIELD), R4.2, R7.2, R8.2, R9.2, U1.15 (DCDC_GND), U1.9 (GND), U3.8 (GND), U3.9 (GND)
